Commit message: Added ros controller for head joint

File: simulation/urdf/robot.xacro (robot description, xacro)
@@ -156,8 +156,19 @@
 	    <axis xyz="0 0 1" />
 	    <origin xyz="0 0 0.08" rpy="0 0 0"/>
-      <limit lower="-3.1416" upper="3.1416" effort="10" velocity="3"/>
+      <limit effort="1000.0" lower="-3.14" upper="3.14" velocity="0.2"/>
+      <hardwareInterface>EffortJointInterface</hardwareInterface>
 	    <parent link="link_neck"/>
 	    <child link="link_head"/>
 	 </joint>
+  <transmission name="head_joint_tran">
+    <type>transmission_interface/SimpleTransmission</type>
+    <joint name="head_joint">
+      <hardwareInterface>EffortJointInterface</hardwareInterface>
+    </joint>
+    <actuator name="motor1">
+      <hardwareInterface>EffortJointInterface</hardwareInterface>
+      <mechanicalReduction>1</mechanicalReduction>
+    </actuator>
+  </transmission>
  <link name="camera_link"> ->
 	    <collision>

Commit message: Updated readme. Added comments

File: simulation/urdf/robot.xacro (robot description, xacro)
@@ -2,18 +2,22 @@
 <robot xmlns:xacro="http://www.ros.org/wiki/xacro" name="robot_xacro">
 <xacro:include filename="$(find simulation)/urdf/robot.gazebo"/>
+  <!-- Wheels properties -->
 	<xacro:property name="length_wheel" value="0.04" />
 	<xacro:property name="radius_wheel" value="0.1" />
+  <!-- Inertia -->
 	<xacro:macro name="default_inertial" params="mass">
-               <inertial>
-                       <mass value="${mass}" />
-                       <origin rpy="0 1.5707 1.5707" xyz="0 0 0"/>
-                       <inertia ixx="0.000526666666667" ixy="0" ixz="0" iyy="0.000526666666667" iyz="0" izz="0.001"/>
-               </inertial>
+  <inertial>
+    <mass value="${mass}" />
+    <origin rpy="0 1.5707 1.5707" xyz="0 0 0"/>
+    <inertia ixx="0.000526666666667" ixy="0" ixz="0" iyy="0.000526666666667" iyz="0" izz="0.001"/>
+  </inertial>
 	</xacro:macro>
-    <xacro:macro name="wheel_geometry">
-		<geometry>
-       			<cylinder length="${length_wheel}" radius="${radius_wheel}"/>
-     	</geometry>
-	</xacro:macro>
+  <!-- Wheels geometry -->
+  <xacro:macro name="wheel_geometry">
+    <geometry>
+      <cylinder length="${length_wheel}" radius="${radius_wheel}"/>
+    </geometry>
+  </xacro:macro>
+	<!-- Materials -->
   <material name="black">
     <color rgba="0.0 0.0 0.0 1.0"/>
@@ -40,4 +44,5 @@
     <color rgba="1.0 1.0 1.0 1.0"/>
   </material>
+<!-- Chassis link -->
 <link name="link_chassis">
   <!-- pose and inertial -->
@@ -75,4 +80,5 @@
   </visual>
 </link>
+<!-- Right wheel link -->
 <link name="link_right_wheel">
   <xacro:default_inertial mass="0.2"/>
@@ -87,4 +93,5 @@
   </visual>
 </link>
+<!-- Left wheel link -->
 <link name="link_left_wheel">
   <xacro:default_inertial mass="0.2"/>
@@ -99,4 +106,5 @@
   </visual>
 </link>
+<!-- Neck link -->
 <link name="link_neck">
   <xacro:default_inertial mass="0.2"/>
@@ -115,4 +123,5 @@
   </visual>
 </link>
+<!-- Head link -->
 <link name="link_head">
   <xacro:default_inertial mass="0.2"/>
@@ -131,4 +140,5 @@
   </visual>
 </link>
+  <!-- Right wheel joint -->
   <joint name="joint_right_wheel" type="continuous">
     <origin rpy="0 0 0" xyz="-0.05 0.15 0"/>
@@ -139,4 +149,5 @@
     <joint_properties damping="1.0" friction="1.0"/>
   </joint>
+  <!-- Left wheel joint -->
   <joint name="joint_left_wheel" type="continuous">
     <origin rpy="0 0 0" xyz="-0.05 -0.15 0"/>
@@ -147,4 +158,5 @@
     <joint_properties damping="1.0" friction="1.0"/>
   </joint>
+  <!-- Neck joint -->
   <joint name="neck_joint" type="fixed">
 	    <axis xyz="0 1 0" />
@@ -153,4 +165,5 @@
 	    <child link="link_neck"/>
 	 </joint>
+  <!-- Head joint -->
    <joint name="head_joint" type="revolute">
 	    <axis xyz="0 0 1" />
@@ -161,4 +174,5 @@
 	    <child link="link_head"/>
 	 </joint>
+  <!-- Transmission for head joint (used to control the joint) -->
   <transmission name="head_joint_tran">
     <type>transmission_interface/SimpleTransmission</type>
@@ -171,4 +185,5 @@
     </actuator>
   </transmission>
+  <!-- Camera link -->
  <link name="camera_link"> ->
 	    <collision>
@@ -193,4 +208,5 @@
 	    </inertial>
   </link>
+  <!-- Camera joint -->
   <joint name="camera_joint" type="fixed">
 	    <axis xyz="0 1 0" />
